File: hardware/main-board/lb-main.sch (KiCad schematic (older format))
At the start: 16 parts, among them IC1 ATMEGA32U4, P1 CONN_4, SW1 SW_PUSH, U1 MICRO-B_USB, X1 CRYSTAL

Commit message: Added a slim version of led light board and controller
Parts:
- added CON1: AVR-ISP-6, AVR-ISP-6, symbol AVR-ISP-6
Connections:
- net labels added: MISO, MOSI, RST, SCK
- wire segments 95 -> 108
- no-connect marks 27 -> 22
Changed lines of the file:
@@
-EESchema Schematic File Version 2  date Sun 05 Jan 2014 02:24:22 PM CET
+EESchema Schematic File Version 2  date Fri 17 Jan 2014 11:20:30 AM CET
 LIBS:power
 LIBS:device
@@
 LIBS:open-project
 LIBS:ws2812b
+LIBS:opendous
+LIBS:FlyingBone-cache
 LIBS:lb-main-cache
 EELAYER 25  0
@@
 Sheet 1 1
 Title ""
-Date "5 jan 2014"
+Date "17 jan 2014"
 Rev ""
 Comp ""
@@
 Comment4 ""
 $EndDescr
+Text GLabel 2950 3800 0    60   Input ~ 0
+SCK
+Text GLabel 2950 3700 0    60   Input ~ 0
+MOSI
+Text GLabel 2950 3600 0    60   Input ~ 0
+MISO
+Text GLabel 5250 1100 0    60   Input ~ 0
+RST
+Text GLabel 5250 900  0    60   Input ~ 0
+MISO
+Text GLabel 5250 1000 0    60   Input ~ 0
+SCK
+Text GLabel 6300 1000 2    60   Input ~ 0
+MOSI
+Wire Wire Line
+	6350 750  6350 900
+Wire Wire Line
+	6350 900  5900 900
+Wire Wire Line
+	3250 1150 3250 1650
+Wire Wire Line
+	3250 1650 3300 1650
+Wire Wire Line
+	3300 3700 2950 3700
+Wire Wire Line
+	5900 1100 6300 1100
+Wire Wire Line
+	5600 1000 5250 1000
 Wire Wire Line
 	6800 3650 7000 3650
 Wire Wire Line
-	7000 3650 7000 4100
+	7000 4100 7000 3650
 Wire Wire Line
 	7000 4100 6350 4100
@@
 Connection ~ 4050 4450
 Wire Wire Line
-	4200 4450 4050 4450
+	4050 4450 4200 4450
 Wire Wire Line
 	1900 2050 2200 2050
@@
 Connection ~ 2450 700
 Wire Wire Line
-	2100 1300 2100 700
-Wire Wire Line
-	2100 700  3050 700
+	2100 700  2100 1300
+Wire Wire Line
+	3050 700  2100 700
 Connection ~ 2450 1200
 Wire Wire Line
@@
 Connection ~ 4450 4350
 Wire Wire Line
-	4050 4350 4600 4350
+	4600 4350 4050 4350
 Wire Wire Line
 	4600 4350 4600 4150
@@
 Connection ~ 3200 2650
 Wire Wire Line
-	3200 2650 3200 2550
+	3200 2550 3200 2650
 Wire Wire Line
 	3200 2550 3300 2550
@@
 	8650 3400 8600 3400
 Wire Wire Line
-	7600 4400 7300 4400
-Wire Wire Line
-	7300 4400 7300 1000
+	7300 4400 7600 4400
+Wire Wire Line
+	7300 1000 7300 4400
 Wire Wire Line
 	7300 3400 7600 3400
@@
 	2700 2150 1900 2150
 Wire Wire Line
-	3300 2650 2100 2650
+	2100 2650 3300 2650
 Wire Wire Line
 	3300 2850 2200 2850
@@
 	2200 2850 2200 3050
 Wire Wire Line
-	2100 2650 2100 1900
+	2100 1900 2100 2650
 Connection ~ 2100 2050
 Wire Wire Line
-	4400 1350 4400 1200
-Wire Wire Line
-	4400 1200 4100 1200
+	4400 1200 4400 1350
+Wire Wire Line
+	4100 1200 4400 1200
 Wire Wire Line
 	4200 1350 4200 1200
@@
 	5950 4950 6400 4950
 Wire Wire Line
-	3300 1850 3050 1850
-Wire Wire Line
-	3050 1850 3050 1100
+	3050 1850 3300 1850
+Wire Wire Line
+	3050 1100 3050 1850
 Connection ~ 3050 1200
 Wire Wire Line
@@
 Connection ~ 6450 4100
 Connection ~ 6650 4100
+Wire Wire Line
+	5600 900  5250 900
+Wire Wire Line
+	5600 1100 5250 1100
+Wire Wire Line
+	5900 1000 6300 1000
+Wire Wire Line
+	3300 3600 2950 3600
+Wire Wire Line
+	3300 3800 2950 3800
+Wire Wire Line
+	6300 1100 6300 1250
 $Comp
 L GND #PWR01
+U 1 1 52D90226
+P 6300 1250
+F 0 "#PWR01" H 6300 1250 30  0001 C CNN
+F 1 "GND" H 6300 1180 30  0001 C CNN
+	1    6300 1250
+	1    0    0    -1
+$EndComp
+$Comp
+L VCC #PWR02
+U 1 1 52D9021A
+P 6350 750
+F 0 "#PWR02" H 6350 850 30  0001 C CNN
+F 1 "VCC" H 6350 850 30  0000 C CNN
+	1    6350 750
+	1    0    0    -1
+$EndComp
+Text Label 3250 1250 0    60   ~ 0
+RST
+Text Label 6200 1100 0    60   ~ 0
+GND
+Text Label 6150 900  0    60   ~ 0
+VCC
+$Comp
+L AVR-ISP-6 CON1
+U 1 1 52D900AF
+P 5750 1000
+F 0 "CON1" H 5670 1240 50  0000 C CNN
+F 1 "AVR-ISP-6" H 5510 770 50  0000 L BNN
+F 2 "AVR-ISP-6" V 5230 1040 50  0001 C CNN
+	1    5750 1000
+	1    0    0    -1
+$EndComp
+$Comp
+L GND #PWR03
 U 1 1 52AEF061
 P 1950 1300
-F 0 "#PWR01" H 1950 1300 30  0001 C CNN
+F 0 "#PWR03" H 1950 1300 30  0001 C CNN
 F 1 "GND" H 1950 1230 30  0001 C CNN
 	1    1950 1300
@@
 $EndComp
 $Comp
-L GND #PWR02
+L GND #PWR04
 U 1 1 52AEF04D
 P 4200 4500
-F 0 "#PWR02" H 4200 4500 30  0001 C CNN
+F 0 "#PWR04" H 4200 4500 30  0001 C CNN
 F 1 "GND" H 4200 4430 30  0001 C CNN
 	1    4200 4500
@@
 $EndComp
 $Comp
-L VCC #PWR03
+L VCC #PWR05
 U 1 1 52AEF035
 P 5700 2900
-F 0 "#PWR03" H 5700 3000 30  0001 C CNN
+F 0 "#PWR05" H 5700 3000 30  0001 C CNN
 F 1 "VCC" H 5700 3000 30  0000 C CNN
 	1    5700 2900
@@
 $EndComp
 $Comp
-L VCC #PWR04
+L VCC #PWR06
 U 1 1 52AEF015
 P 2200 1900
-F 0 "#PWR04" H 2200 2000 30  0001 C CNN
+F 0 "#PWR06" H 2200 2000 30  0001 C CNN
 F 1 "VCC" H 2200 2000 30  0000 C CNN
 	1    2200 1900
@@
 $EndComp
 $Comp
-L VCC #PWR05
+L VCC #PWR07
 U 1 1 52AEEFE5
 P 7450 1350
-F 0 "#PWR05" H 7450 1450 30  0001 C CNN
+F 0 "#PWR07" H 7450 1450 30  0001 C CNN
 F 1 "VCC" H 7450 1450 30  0000 C CNN
 	1    7450 1350
@@
 NoConn ~ 5200 1650
 NoConn ~ 1900 2350
-NoConn ~ 3300 1650
-NoConn ~ 5250 1650
 NoConn ~ 5200 1750
 NoConn ~ 5200 1900
@@
 NoConn ~ 5200 3850
 NoConn ~ 3300 3900
-NoConn ~ 3300 3800
-NoConn ~ 3300 3700
-NoConn ~ 3300 3600
 NoConn ~ 3300 3500
 NoConn ~ 3300 3400
@@
 NoConn ~ 3300 3200
 $Comp
-L VCC #PWR06
+L VCC #PWR08
 U 1 1 52AEEF4C
 P 5600 2900
-F 0 "#PWR06" H 5600 3000 30  0001 C CNN
+F 0 "#PWR08" H 5600 3000 30  0001 C CNN
 F 1 "VCC" H 5600 3000 30  0000 C CNN
 	1    5600 2900
@@
 $EndComp
 $Comp
-L GND #PWR07
+L GND #PWR09
 U 1 1 52AE325C
 P 2100 1300
-F 0 "#PWR07" H 2100 1300 30  0001 C CNN
+F 0 "#PWR09" H 2100 1300 30  0001 C CNN
 F 1 "GND" H 2100 1230 30  0001 C CNN
 	1    2100 1300
@@
 $EndComp
 $Comp
-L GND #PWR08
+L GND #PWR010
 U 1 1 52AE30FE
 P 6500 4150
-F 0 "#PWR08" H 6500 4150 30  0001 C CNN
+F 0 "#PWR010" H 6500 4150 30  0001 C CNN
 F 1 "GND" H 6500 4080 30  0001 C CNN
 	1    6500 4150
@@
 $EndComp
 $Comp
-L VCC #PWR09
+L VCC #PWR011
 U 1 1 52AE30ED
 P 6100 3000
-F 0 "#PWR09" H 6100 3100 30  0001 C CNN
+F 0 "#PWR011" H 6100 3100 30  0001 C CNN
 F 1 "VCC" H 6100 3100 30  0000 C CNN
 	1    6100 3000
@@
 $EndComp
 $Comp
-L VCC #PWR010
+L VCC #PWR012
 U 1 1 52ADE4F1
 P 4100 1050
-F 0 "#PWR010" H 4100 1150 30  0001 C CNN
+F 0 "#PWR012" H 4100 1150 30  0001 C CNN
 F 1 "VCC" H 4100 1150 30  0000 C CNN
 	1    4100 1050
@@
 $EndComp
 $Comp
-L GND #PWR011
+L GND #PWR013
 U 1 1 52ADE4E8
 P 4050 4500
-F 0 "#PWR011" H 4050 4500 30  0001 C CNN
+F 0 "#PWR013" H 4050 4500 30  0001 C CNN
 F 1 "GND" H 4050 4430 30  0001 C CNN
 	1    4050 4500
@@
 $EndComp
 $Comp
-L VCC #PWR012
+L VCC #PWR014
 U 1 1 52ADE420
 P 6300 4750
-F 0 "#PWR012" H 6300 4850 30  0001 C CNN
+F 0 "#PWR014" H 6300 4850 30  0001 C CNN
 F 1 "VCC" H 6300 4850 30  0000 C CNN
 	1    6300 4750
@@
 $EndComp
 $Comp
-L VCC #PWR013
+L VCC #PWR015
 U 1 1 52ADE418
 P 7300 1000
-F 0 "#PWR013" H 7300 1100 30  0001 C CNN
+F 0 "#PWR015" H 7300 1100 30  0001 C CNN
 F 1 "VCC" H 7300 1100 30  0000 C CNN
 	1    7300 1000
@@
 $EndComp
 $Comp
-L VCC #PWR014
+L VCC #PWR016
 U 1 1 52ADE408
 P 2100 1900
-F 0 "#PWR014" H 2100 2000 30  0001 C CNN
+F 0 "#PWR016" H 2100 2000 30  0001 C CNN
 F 1 "VCC" H 2100 2000 30  0000 C CNN
 	1    2100 1900
@@
 $EndComp
 $Comp
-L GND #PWR015
+L GND #PWR017
 U 1 1 52ADE3DA
 P 6300 5300
-F 0 "#PWR015" H 6300 5300 30  0001 C CNN
+F 0 "#PWR017" H 6300 5300 30  0001 C CNN
 F 1 "GND" H 6300 5230 30  0001 C CNN
 	1    6300 5300
@@
 $EndComp
 $Comp
-L GND #PWR016
+L GND #PWR018
 U 1 1 52ADE3D3
 P 9000 5000
-F 0 "#PWR016" H 9000 5000 30  0001 C CNN
+F 0 "#PWR018" H 9000 5000 30  0001 C CNN
 F 1 "GND" H 9000 4930 30  0001 C CNN
 	1    9000 5000
@@
 $EndComp
 $Comp
-L GND #PWR017
+L GND #PWR019
 U 1 1 52ADE3C0
 P 2200 3550
-F 0 "#PWR017" H 2200 3550 30  0001 C CNN
+F 0 "#PWR019" H 2200 3550 30  0001 C CNN
 F 1 "GND" H 2200 3480 30  0001 C CNN
 	1    2200 3550
@@
 $EndComp
 $Comp
-L GND #PWR018
+L GND #PWR020
 U 1 1 52ADE3BB
 P 1950 2800
-F 0 "#PWR018" H 1950 2800 30  0001 C CNN
+F 0 "#PWR020" H 1950 2800 30  0001 C CNN
 F 1 "GND" H 1950 2730 30  0001 C CNN
 	1    1950 2800
