File: hardware/slim-light-controller/slim-light-controller.sch (KiCad schematic (older format))
At the start: 17 parts, among them K1 USBCONN, K2 CONN_3, K3 AVR-ISP-6, K4 CONN_2, U1 ATTINY84-SS, X1 16MHz

Commit message: Updated schematics after first test. Added a basic Arduino program without USB functionality.
Parts:
- added R?: 330, symbol R
- R4: value 10k -> 330
Connections:
- wire segments 68 -> 69
Other:
- moved on the sheet: D3, K2, R4
Changed lines of the file:
@@
-EESchema Schematic File Version 2  date Mon 20 Jan 2014 12:27:20 PM CET
+EESchema Schematic File Version 2  date sön  6 apr 2014 12:13:33
 LIBS:power
 LIBS:device
@@
 LIBS:contrib
 LIBS:valves
-LIBS:opendous
-LIBS:avr-isp-6
 LIBS:slim-light-controller-cache
 EELAYER 25  0
@@
 Sheet 1 1
 Title ""
-Date "19 jan 2014"
+Date "6 apr 2014"
 Rev ""
 Comp ""
@@
 $EndDescr
 Wire Wire Line
+	7450 4950 7400 4950
+Wire Wire Line
+	5650 3850 5500 3850
+Wire Wire Line
+	6300 3250 6300 3700
+Wire Wire Line
+	7450 3500 7450 4000
+Wire Wire Line
+	8050 4950 7950 4950
+Wire Wire Line
+	8050 4850 8000 4850
+Wire Wire Line
+	8000 4850 8000 4750
+Wire Wire Line
+	6800 3250 6800 3150
+Wire Wire Line
+	6800 3150 6850 3150
+Wire Wire Line
+	5850 3000 6000 3000
+Wire Wire Line
+	7800 4500 7450 4500
+Wire Wire Line
+	7800 4500 7800 3900
+Wire Wire Line
+	6900 1675 6625 1675
+Wire Wire Line
+	7325 1950 7325 1775
+Wire Wire Line
+	7325 1775 7150 1775
+Connection ~ 6700 5050
+Wire Wire Line
+	6700 5150 6700 5050
+Wire Wire Line
+	6550 4950 6550 5050
+Wire Wire Line
+	6550 5050 6850 5050
+Wire Wire Line
+	6850 5050 6850 4950
+Connection ~ 6550 4000
+Wire Wire Line
+	5500 4050 6000 4050
+Wire Wire Line
+	6000 4050 6000 4000
+Wire Wire Line
+	6000 4000 6850 4000
+Wire Wire Line
+	6550 4550 6550 4400
+Wire Wire Line
+	5500 3750 5550 3750
+Wire Wire Line
+	5500 3550 5550 3550
+Wire Wire Line
+	6300 3250 5500 3250
+Wire Wire Line
+	5500 3150 6250 3150
+Wire Wire Line
+	6300 3700 6850 3700
+Wire Wire Line
+	6850 3600 6250 3600
+Wire Wire Line
+	7350 3600 7900 3600
+Wire Wire Line
+	7450 4500 7450 4400
+Wire Wire Line
+	7900 3700 7350 3700
+Connection ~ 3350 3150
+Wire Wire Line
+	3350 3500 3350 3150
+Connection ~ 3350 4350
+Wire Wire Line
+	3350 3900 3350 4350
+Connection ~ 7800 4000
+Wire Wire Line
+	7800 3900 7900 3900
+Wire Wire Line
+	7750 3300 7750 3800
+Wire Wire Line
+	7750 3800 7900 3800
+Wire Wire Line
+	7900 4000 7800 4000
+Wire Wire Line
+	3400 4350 3200 4350
+Wire Wire Line
+	3200 4350 3200 4550
+Wire Wire Line
+	3400 3150 3200 3150
+Wire Wire Line
+	3200 3150 3200 2900
+Wire Wire Line
+	7600 4000 7600 3600
+Connection ~ 7600 3600
+Wire Wire Line
+	7600 4400 7600 4600
+Connection ~ 7600 4500
+Connection ~ 7450 3700
+Connection ~ 6250 3600
+Wire Wire Line
+	5500 4250 6250 4250
+Wire Wire Line
+	5500 3650 5550 3650
+Wire Wire Line
+	5500 4350 5550 4350
+Wire Wire Line
+	6850 4000 6850 4550
+Wire Wire Line
+	6550 4400 6150 4400
+Wire Wire Line
+	6150 4400 6150 4150
+Wire Wire Line
+	6150 4150 5500 4150
+Wire Wire Line
+	7150 1575 7325 1575
+Wire Wire Line
+	7325 1575 7325 1400
+Wire Wire Line
+	6900 1775 6625 1775
+Wire Wire Line
+	6900 1575 6625 1575
+Wire Wire Line
+	7150 1675 7500 1675
+Wire Wire Line
+	6800 3850 6900 3850
+Wire Wire Line
+	6900 3850 6900 3900
+Wire Wire Line
+	6400 3850 6150 3850
+Wire Wire Line
+	5500 3350 5850 3350
+Wire Wire Line
+	5850 3350 5850 3000
+Wire Wire Line
+	5850 2500 5850 2400
+Wire Wire Line
+	6850 2950 6000 2950
+Wire Wire Line
+	6000 2950 6000 3000
+Wire Wire Line
+	8050 5050 8000 5050
+Wire Wire Line
+	8000 5050 8000 5150
+Wire Wire Line
 	7450 3000 7450 2850
 Wire Wire Line
-	7800 5100 7800 5000
-Wire Wire Line
-	7800 5000 7850 5000
-Wire Wire Line
-	6000 2950 6000 3000
-Wire Wire Line
-	6000 2950 6850 2950
-Wire Wire Line
-	5850 2500 5850 2400
-Wire Wire Line
-	5850 3350 5850 3000
-Wire Wire Line
-	5850 3350 5500 3350
-Wire Wire Line
-	6400 3450 6100 3450
-Wire Wire Line
-	6900 3500 6900 3450
-Wire Wire Line
-	6900 3450 6800 3450
-Wire Wire Line
-	7150 1675 7500 1675
-Wire Wire Line
-	6900 1575 6625 1575
-Wire Wire Line
-	6900 1775 6625 1775
-Wire Wire Line
-	7325 1400 7325 1575
-Wire Wire Line
-	7325 1575 7150 1575
-Wire Wire Line
-	5500 4150 6150 4150
-Wire Wire Line
-	6150 4150 6150 4400
-Wire Wire Line
-	6150 4400 6550 4400
-Wire Wire Line
-	6850 4550 6850 4000
-Wire Wire Line
-	5500 4350 5550 4350
-Wire Wire Line
-	5500 3650 5550 3650
-Wire Wire Line
-	5500 4250 6250 4250
-Wire Wire Line
 	6250 4250 6250 3150
-Connection ~ 6250 3600
-Connection ~ 7450 3700
-Connection ~ 7600 4500
-Wire Wire Line
-	7600 4400 7600 4600
-Connection ~ 7600 3600
-Wire Wire Line
-	7600 4000 7600 3600
-Wire Wire Line
-	3200 2900 3200 3150
-Wire Wire Line
-	3200 3150 3400 3150
-Wire Wire Line
-	3200 4550 3200 4350
-Wire Wire Line
-	3200 4350 3400 4350
-Wire Wire Line
-	7900 4000 7800 4000
-Wire Wire Line
-	7900 3800 7750 3800
-Wire Wire Line
-	7750 3800 7750 3300
-Wire Wire Line
-	7900 3900 7800 3900
-Connection ~ 7800 4000
-Wire Wire Line
-	3350 3900 3350 4350
-Connection ~ 3350 4350
-Wire Wire Line
-	3350 3500 3350 3150
-Connection ~ 3350 3150
-Wire Wire Line
-	7900 3700 7350 3700
-Wire Wire Line
-	7450 4400 7450 4500
-Wire Wire Line
-	7350 3600 7900 3600
-Wire Wire Line
-	6250 3600 6850 3600
-Wire Wire Line
-	6850 3700 6300 3700
-Wire Wire Line
-	6300 3700 6300 3250
-Wire Wire Line
-	6250 3150 5500 3150
-Wire Wire Line
-	6300 3250 5500 3250
-Wire Wire Line
-	5500 3550 5550 3550
-Wire Wire Line
-	5500 3750 5550 3750
-Wire Wire Line
-	6550 4400 6550 4550
-Wire Wire Line
-	6850 4000 6000 4000
-Wire Wire Line
-	6000 4000 6000 4050
-Wire Wire Line
-	6000 4050 5500 4050
-Connection ~ 6550 4000
-Wire Wire Line
-	6850 4950 6850 5050
-Wire Wire Line
-	6850 5050 6550 5050
-Wire Wire Line
-	6550 5050 6550 4950
-Wire Wire Line
-	6700 5050 6700 5150
-Connection ~ 6700 5050
-Wire Wire Line
-	7150 1775 7325 1775
-Wire Wire Line
-	7325 1775 7325 1950
-Wire Wire Line
-	6900 1675 6625 1675
-Wire Wire Line
-	5500 3850 5975 3850
-Wire Wire Line
-	7800 3900 7800 4500
-Wire Wire Line
-	7800 4500 7450 4500
-Wire Wire Line
-	5600 3450 5500 3450
-Wire Wire Line
-	5850 3000 6000 3000
-Wire Wire Line
-	6850 3150 6800 3150
-Wire Wire Line
-	6800 3150 6800 3250
-Wire Wire Line
-	7800 4700 7800 4800
-Wire Wire Line
-	7800 4800 7850 4800
-Wire Wire Line
-	7850 4900 7700 4900
-Wire Wire Line
-	7450 3500 7450 4000
+Wire Wire Line
+	5500 3450 5550 3450
+$Comp
+L R R?
+U 1 1 53412875
+P 7700 4950
+F 0 "R?" V 7780 4950 50  0000 C CNN
+F 1 "330" V 7700 4950 50  0000 C CNN
+	1    7700 4950
+	0    -1   -1   0
+$EndComp
+Text GLabel 5550 3450 2    60   Output ~ 0
+SOUT
 $Comp
 L VCC #PWR01
@@
 L GND #PWR04
 U 1 1 52DBDC82
-P 6900 3500
-F 0 "#PWR04" H 6900 3500 30  0001 C CNN
-F 1 "GND" H 6900 3430 30  0001 C CNN
-	1    6900 3500
+P 6900 3900
+F 0 "#PWR04" H 6900 3900 30  0001 C CNN
+F 1 "GND" H 6900 3830 30  0001 C CNN
+	1    6900 3900
 	1    0    0    -1
 $EndComp
@@
 L LED D3
 U 1 1 52DBDC6F
-P 6600 3450
-F 0 "D3" H 6600 3550 50  0000 C CNN
-F 1 "LED" H 6600 3350 50  0000 C CNN
-	1    6600 3450
+P 6600 3850
+F 0 "D3" H 6600 3950 50  0000 C CNN
+F 1 "LED" H 6600 3750 50  0000 C CNN
+	1    6600 3850
 	1    0    0    -1
 $EndComp
@@
 L R R4
 U 1 1 52DBDC45
-P 5850 3450
-F 0 "R4" V 5930 3450 50  0000 C CNN
-F 1 "10k" V 5850 3450 50  0000 C CNN
-	1    5850 3450
+P 5900 3850
+F 0 "R4" V 5980 3850 50  0000 C CNN
+F 1 "330" V 5900 3850 50  0000 C CNN
+	1    5900 3850
 	0    -1   -1   0
 $EndComp
@@
 L VCC #PWR05
 U 1 1 52DA86C6
-P 7800 4700
-F 0 "#PWR05" H 7800 4800 30  0001 C CNN
-F 1 "VCC" H 7800 4800 30  0000 C CNN
-	1    7800 4700
+P 8000 4750
+F 0 "#PWR05" H 8000 4850 30  0001 C CNN
+F 1 "VCC" H 8000 4850 30  0000 C CNN
+	1    8000 4750
 	1    0    0    -1
 $EndComp
@@
 L GND #PWR06
 U 1 1 52DA86BE
-P 7800 5100
-F 0 "#PWR06" H 7800 5100 30  0001 C CNN
-F 1 "GND" H 7800 5030 30  0001 C CNN
-	1    7800 5100
-	1    0    0    -1
-$EndComp
-Text GLabel 7700 4900 0    60   Input ~ 0
+P 8000 5150
+F 0 "#PWR06" H 8000 5150 30  0001 C CNN
+F 1 "GND" H 8000 5080 30  0001 C CNN
+	1    8000 5150
+	1    0    0    -1
+$EndComp
+Text GLabel 7400 4950 0    60   Input ~ 0
 SOUT
 $Comp
 L CONN_3 K2
 U 1 1 52DA86A5
-P 8200 4900
-F 0 "K2" V 8150 4900 50  0000 C CNN
-F 1 "CONN_3" V 8250 4900 40  0000 C CNN
-	1    8200 4900
+P 8400 4950
+F 0 "K2" V 8350 4950 50  0000 C CNN
+F 1 "CONN_3" V 8450 4950 40  0000 C CNN
+	1    8400 4950
 	1    0    0    1
 $EndComp
-Text GLabel 5975 3850 2    60   Input ~ 0
-SOUT
 $Comp
 L VCC #PWR07
